File: 1RGBLed.kicad_sch (KiCad schematic)
At the start: 10 parts, among them J1 JST_SH_SM06B-SRSS-TB_1x06-1MP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, J4 Conn_01x04, U1 M24C02-FMN, U2 LP5815DRLR

Commit message: Update MNP for the LED and the driver
Parts:
- D1: Feeder (none) -> 8mm; MPN (none) -> C458749
- U2: Feeder (none) -> 8mm; MPN (none) -> C47262831
Changed lines of the file:
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@@
 			)
 		)
-		(property "MPN" ""
+		(property "MPN" "C47262831"
 			(at 44.45 31.75 0)
 			(effects
@@
 			)
 		)
-		(property "Feeder" ""
+		(property "Feeder" "8mm"
 			(at 44.45 31.75 0)
 			(effects
@@
 			(at 95.25 36.83 0)
 			(effects
+				(font
+					(size 1.27 1.27)
+				)
+				(hide yes)
+			)
+		)
+		(property "MPN" "C458749"
+			(at 95.25 36.83 0)
+			(effects
+				(font
+					(size 1.27 1.27)
+				)
+				(hide yes)
+			)
+		)
+		(property "Feeder" "8mm"
+			(at 95.25 36.83 0)
+			(effects
